Commit message: up

File: pbot-jackal_description/urdf/pbot_jackal.urdf.xacro (robot description, xacro)
@@ -1,5 +1,11 @@
 <?xml version="1.0"?>
 <robot name="pbot-jackal" xmlns:xacro="http://www.ros.org/wiki/xacro">
-    <!-- Include the base robot model -->
-    <xacro:include filename="$(find jackal_description)/urdf/jackal.urdf.xacro" />
+  <!-- Include the base robot model -->
+  <xacro:include filename="$(find jackal_description)/urdf/jackal.urdf.xacro" />
+  <link name="velodyne_vlp16"></link>
+  <joint name="velodyne_vlp16_joint" type="fixed">
+    <parent link="mid_mount" />
+    <child link="velodyne_mount" />
+    <origin xyz="0.09 0 0" />
+  </joint>
 </robot>
