Commit message: up

File: pbot-jackal_description/urdf/pbot_jackal_additional_parts.urdf.xacro (robot description, xacro)
@@ -3,9 +3,21 @@
        by setting the JACKAL_URDF_EXTRAS environment variable to the full
        path of this file. -->
+  <link name="front_laser"></link>
+  <joint name="front_laser_joint" type="fixed">
+    <parent link="front_mount" />
+    <child link="front_laser" />
+    <origin xyz="0.1 0 0.53" rpy="0 0 0"/>
+  </joint>
   <link name="velodyne_vlp16_mount"></link>
   <joint name="velodyne_vlp16_mount_joint" type="fixed">
-    <parent link="front_mount" />
+    <parent link="front_laser" />
     <child link="velodyne_vlp16_mount" />
-    <origin xyz="-0.03 0 0" rpy="0 0 0"/>
+    <origin xyz="0 0 0" rpy="0 0 0"/>
+  </joint>
+  <link name="velodyne"></link>
+  <joint name="velodyne_joint" type="fixed">
+    <parent link="velodyne_vlp16_mount" />
+    <child link="velodyne" />
+    <origin xyz="0 0 0" rpy="0 0 0"/>
   </joint>
 </robot>
